File: bite force sens.kicad_sch (KiCad schematic)
At the start: 21 parts, among them J1 Flexiforce, J2 oled display, J4 switch, J6 Conn_01x02, J7 Conn_01x02, U1 XIAO ESP32 S3, U2 MCP6004

Commit message: Update bite force sens.kicad_sch
Other:
- title: bite force sensor -> bfs
Changed lines of the file:
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@@
 	(paper "A4")
 	(title_block
-		(title "bite force sensor")
+		(title "bfs")
 		(date "15-04-2025")
 		(company "Varidhi educational products")
