File: bite force sens.kicad_sch (KiCad schematic)
At the start: 19 parts, among them J1 Flexiforce, J2 oled display, J4 switch, J6 Conn_01x02, J7 Conn_01x02, U1 XIAO ESP32 S3, U2 MCP6004

Commit message: made entire change in design and now the fresh pcb will be done and comitted at next commit
Parts:
- removed D1, D2: 1N5711UR, Diode_SMD:D_MELF, symbol Diode:1N5711UR
- removed J1: Flexiforce, Connector:FanPinHeader_1x03_P2.54mm_Vertical, symbol Connector_Generic:Conn_01x03
- removed J2: oled display, Connector:FanPinHeader_1x04_P2.54mm_Vertical, symbol Connector_Generic:Conn_01x04
- removed J4: switch, Connector:FanPinHeader_1x03_P2.54mm_Vertical, symbol Connector_Generic:Conn_01x03
- removed J6, J7: Conn_01x02, Connector_JST:JST_XH_S2B-XH-A-1_1x02_P2.50mm_Horizontal, symbol Connector_Generic:Conn_01x02
- removed U1: XIAO ESP32 S3, XIAO_Footprints:MODULE_102010428, symbol 102010428:102010428
- removed U2: MCP6004, Package_SO:SOIC-14_3.9x8.7mm_P1.27mm, symbol Amplifier_Operational:MCP6004
- added C10: 10u, Capacitor_SMD:C_0805_2012Metric, symbol Device:C
- added C11, C7: 47p, Capacitor_SMD:C_0805_2012Metric, symbol Device:C
- added C14: C, Capacitor_SMD:C_0805_2012Metric, symbol Device:C
- added C15: 0.1u, Capacitor_SMD:C_0805_2012Metric, symbol Device:C
- added D1, D2, D4: D_Schottky, Diode_SMD:D_SMA, symbol Device:D_Schottky
- added D3: D_Zener, Diode_SMD:D_SMA, symbol Device:D_Zener
- added J1: lipo bat, Connector_AMASS:AMASS_XT30PW-M_1x02_P2.50mm_Horizontal, symbol Connector:Conn_01x02_Socket
- added J2, J3: tp4056 pin, Connector_PinHeader_2.54mm:PinHeader_1x02_P2.54mm_Vertical, symbol Connector:Conn_01x02_Pin
- added J4: fsr, Connector_JST:JST_PH_B2B-PH-K_1x02_P2.00mm_Vertical, symbol Connector:Conn_01x02_Socket
- added J5: display, connec:Hirose_FH12-8S-0.5SH_1x08-1MP_P0.50mm_Horizontal, symbol Connector:Conn_01x08_Socket
- added R9: 100k, Resistor_SMD:R_0805_2012Metric, symbol Device:R
- added SW1: on/off, Button_Switch_SMD:SW_DIP_SPSTx01_Slide_6.7x4.1mm_W6.73mm_P2.54mm_LowProfile_JPin, symbol Switch:SW_SPST
- added SW2: reset, Button_Switch_THT:SW_PUSH_6mm, symbol Switch:SW_Push
- added U1: MCP6004, Package_SO:SOIC-14_3.9x8.7mm_P1.27mm, symbol Amplifier_Operational:MCP6004
- added U2: MCP1700-3302E_TO, mcp1700:TO127P254X495-3, symbol MCP1700-3302E_TO:MCP1700-3302E_TO
- added U3: ESP32-C3-WROOM-02-N4, esp32 footrpint:MODULE_ESP32-C3-WROOM-02-H4, symbol ESP32-C3-WROOM-02-N4:ESP32-C3-WROOM-02-N4
- C1, C2: value 47p -> 10u; footprint Capacitor_SMD:C_0603_1608Metric -> Capacitor_SMD:C_0805_2012Metric
- C3, C4: footprint Capacitor_SMD:C_0603_1608Metric -> Capacitor_SMD:C_0805_2012Metric
- R1: value 80k -> 20k; footprint Resistor_SMD:R_0603_1608Metric_Pad0.98x0.95mm_HandSolder -> Resistor_SMD:R_0805_2012Metric
- R2: value 20k -> 80k; footprint Resistor_SMD:R_0603_1608Metric_Pad0.98x0.95mm_HandSolder -> Resistor_SMD:R_0805_2012Metric
- R3: value 100k -> 10k; footprint Resistor_SMD:R_0603_1608Metric_Pad0.98x0.95mm_HandSolder -> Resistor_SMD:R_0805_2012Metric
- R4, R6: footprint Resistor_SMD:R_0603_1608Metric_Pad0.98x0.95mm_HandSolder -> Resistor_SMD:R_0805_2012Metric
- R5: value 10k -> 33; footprint Resistor_SMD:R_0603_1608Metric_Pad0.98x0.95mm_HandSolder -> Resistor_SMD:R_0805_2012Metric
Connections:
- net 3v3: now also C4.2, R2.1, R4.2, R5.2, C10.2, C14.1, C15.2, D4.1 (K), J5.7 (Pin_7), SW1.2 (B), U1.4 (V+), U3.1 (3V3); no longer C3.2, R1.1, R6.2
- net GND: now also C1.1, C2.2, R1.2, R6.1, C10.1, C14.2, C15.1, C7.2, D1.2 (A), D2.2 (A), D3.2 (A), J3.1 (Pin_1), J4.2 (Pin_2), J5.2 (Pin_2), SW2.2, U1.11 (V-), U2.1 (GND), U3.19 (GND__1), U3.20 (GND__2), U3.21 (GND__3), U3.22 (GND__4), U3.23 (GND__5), U3.24 (GND__6), U3.25 (GND__7), U3.26 (GND__8), U3.27 (GND__9), U3.28 (GND__10), U3.29 (GND__11), U3.30 (GND__12), U3.31 (GND__13), U3.32 (GND__14), U3.33 (GND__15), U3.34 (GND__16), U3.35 (GND__17), U3.36 (GND__18), U3.37 (GND__19), U3.38 (GND__20), U3.39 (GND__21), U3.9 (GND); no longer C2.1, R2.2, R5.2
- net at R5.1: now also J5.1 (Pin_1); no longer R6.1
- net v2: now reaches R3.1
- net v2: now also C11.2, R9.2, U1.7; no longer C1.1
- new net: C7.1, R3.2, U1.10 (+)
- new net: C11.1, J4.1 (Pin_1), R9.1, U1.6 (-)
- new net: R4.1, R6.2, U1.12 (+)
- new net: U1.13 (-), U1.14
- new net +: D2.1 (K), J1.2 (Pin_2), J2.2 (Pin_2)
- new net -: J1.1 (Pin_1), J3.2 (Pin_2)
- new net 3.3: C2.1, SW1.1 (A), U2.3 (VOUT)
- new net CS: J5.8 (Pin_8), U3.10 (IO10)
- new net RESET: J5.3 (Pin_3), U3.7 (IO8)
- new net RS: J5.4 (Pin_4), U3.8 (IO9)
- new net SCL: J5.6 (Pin_6), U3.5 (IO6)
- new net SDA: J5.5 (Pin_5), U3.6 (IO7)
- new net V3: D1.1 (K), D4.2 (A), U1.8, U1.9 (-), U3.15 (IO3)
- new net en: SW2.1, U3.2 (EN)
- new net v: C1.2, C3.2, D3.1 (K), J2.1 (Pin_1), U2.2 (VIN)
- new net v0: R1.1, R2.2, U1.3 (+)
- new net v1: U1.1, U1.2 (-), U1.5 (+)
- no-connect marks 7 -> 9
Other:
- title: bfs -> BITE FORCE SENSORY SYSTEM

Commit message: completed the pcb design
Parts:
- C14: value C -> 0.1u
- J1: footprint Connector_AMASS:AMASS_XT30PW-M_1x02_P2.50mm_Horizontal -> Connector:JWT_A3963_1x02_P3.96mm_Vertical
- U3: footprint esp32 footrpint:MODULE_ESP32-C3-WROOM-02-H4 -> Library:MODULE_ESP32-C3-WROOM-02-H4
Changed lines of the file:
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@@
 			)
 		)
-		(property "Value" "C"
+		(property "Value" "0.1u"
 			(at 185.42 99.06 90)
 			(effects
@@
 			)
 		)
-		(property "Footprint" "esp32 footrpint:MODULE_ESP32-C3-WROOM-02-H4"
+		(property "Footprint" "Library:MODULE_ESP32-C3-WROOM-02-H4"
 			(at 228.6 57.15 0)
 			(effects
@@
 			)
 		)
-		(property "Footprint" "Connector_AMASS:AMASS_XT30PW-M_1x02_P2.50mm_Horizontal"
+		(property "Footprint" "Connector:JWT_A3963_1x02_P3.96mm_Vertical"
 			(at 26.67 57.15 0)
 			(effects
